File: obs_avoidance/schematics/Ultrasonics/Ultrasonics.sch (EAGLE design)
At the start: 6 parts

Commit message: Added DC-DC converter to the board
Parts:
- removed BATTERY_HEADERS: 5V, pinhead:PINHD-1X2
- added U$2: DC-DC-STEP-DOWN-LM2596, diy-modules:DC-DC-STEP-DOWN-LM2596
Connections:
- net N$1: now also U$2.OUT+; no longer BATTERY_HEADERS.1
- net N$10: now also U$2.OUT-; no longer BATTERY_HEADERS.2
Changed lines of the file:
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@@
 <layer number="97" name="Info" color="7" fill="1" visible="yes" active="yes"/>
 <layer number="98" name="Guide" color="6" fill="1" visible="yes" active="yes"/>
+<layer number="101" name="Hidden" color="15" fill="1" visible="yes" active="yes"/>
+<layer number="102" name="Changes" color="12" fill="1" visible="yes" active="yes"/>
 </layers>
 <schematic xreflabel="%F%N/%S.%C%R" xrefpart="/%S.%C%R">
@@
 <part name="JSN-SR04T_3" library="pinhead" library_urn="urn:adsk.eagle:library:325" deviceset="PINHD-1X4" device="" package3d_urn="urn:adsk.eagle:package:22407/2"/>
 <part name="JSN-SR04T_4" library="pinhead" library_urn="urn:adsk.eagle:library:325" deviceset="PINHD-1X4" device="" package3d_urn="urn:adsk.eagle:package:22407/2"/>
-<part name="BATTERY_HEADERS" library="pinhead" library_urn="urn:adsk.eagle:library:325" deviceset="PINHD-1X2" device="" package3d_urn="urn:adsk.eagle:package:22435/2" value="5V"/>
+<part name="U$2" library="diy-modules" deviceset="DC-DC-STEP-DOWN-LM2596" device=""/>
 </parts>
 <sheets>
@@
 <attribute name="VALUE" x="-35.56" y="39.37" size="1.778" layer="96" rot="R90"/>
 </instance>
-<instance part="BATTERY_HEADERS" gate="G$1" x="22.86" y="40.64" smashed="yes">
-<attribute name="NAME" x="16.51" y="46.355" size="1.778" layer="95"/>
-<attribute name="VALUE" x="16.51" y="35.56" size="1.778" layer="96"/>
+<instance part="U$2" gate="G$1" x="149.86" y="33.02" smashed="yes" rot="MR0">
+<attribute name="NAME" x="162.56" y="48.26" size="1.778" layer="95" rot="MR0"/>
+<attribute name="VALUE" x="162.56" y="45.72" size="1.778" layer="96" rot="MR0"/>
 </instance>
 </instances>
@@
 <wire x1="30.48" y1="43.18" x2="35.56" y2="43.18" width="0.1524" layer="91"/>
 <wire x1="35.56" y1="43.18" x2="35.56" y2="48.26" width="0.1524" layer="91"/>
-<junction x="30.48" y="43.18"/>
-<pinref part="BATTERY_HEADERS" gate="G$1" pin="1"/>
-<wire x1="20.32" y1="43.18" x2="12.7" y2="43.18" width="0.1524" layer="91"/>
-<wire x1="12.7" y1="43.18" x2="12.7" y2="50.8" width="0.1524" layer="91"/>
-<wire x1="12.7" y1="50.8" x2="30.48" y2="50.8" width="0.1524" layer="91"/>
-<wire x1="30.48" y1="50.8" x2="30.48" y2="43.18" width="0.1524" layer="91"/>
 <pinref part="JSN-SR04T_3" gate="A" pin="1"/>
 <wire x1="-20.32" y1="68.58" x2="-27.94" y2="68.58" width="0.1524" layer="91"/>
@@
 <wire x1="-53.34" y1="78.74" x2="-48.26" y2="78.74" width="0.1524" layer="91"/>
 <wire x1="-48.26" y1="78.74" x2="-48.26" y2="101.6" width="0.1524" layer="91"/>
+<wire x1="30.48" y1="-7.62" x2="111.76" y2="-7.62" width="0.1524" layer="91"/>
+<wire x1="111.76" y1="-7.62" x2="111.76" y2="38.1" width="0.1524" layer="91"/>
+<junction x="30.48" y="-7.62"/>
+<pinref part="U$2" gate="G$1" pin="OUT+"/>
+<wire x1="111.76" y1="38.1" x2="132.08" y2="38.1" width="0.1524" layer="91"/>
 </segment>
 </net>
@@
 <wire x1="-93.98" y1="60.96" x2="-93.98" y2="-2.54" width="0.1524" layer="91"/>
 <wire x1="-93.98" y1="-2.54" x2="38.1" y2="-2.54" width="0.1524" layer="91"/>
-<wire x1="38.1" y1="-2.54" x2="38.1" y2="40.64" width="0.1524" layer="91"/>
-<wire x1="38.1" y1="40.64" x2="35.56" y2="40.64" width="0.1524" layer="91"/>
-<wire x1="35.56" y1="40.64" x2="33.02" y2="40.64" width="0.1524" layer="91"/>
+<wire x1="38.1" y1="27.94" x2="38.1" y2="40.64" width="0.1524" layer="91"/>
+<wire x1="38.1" y1="40.64" x2="33.02" y2="40.64" width="0.1524" layer="91"/>
 <wire x1="-88.9" y1="60.96" x2="-88.9" y2="93.98" width="0.1524" layer="91"/>
 <wire x1="-88.9" y1="93.98" x2="-38.1" y2="93.98" width="0.1524" layer="91"/>
@@
 <pinref part="U$1" gate="G$1" pin="GND"/>
 <wire x1="33.02" y1="50.8" x2="35.56" y2="50.8" width="0.1524" layer="91"/>
-<pinref part="BATTERY_HEADERS" gate="G$1" pin="2"/>
-<wire x1="20.32" y1="40.64" x2="12.7" y2="40.64" width="0.1524" layer="91"/>
-<wire x1="12.7" y1="40.64" x2="12.7" y2="35.56" width="0.1524" layer="91"/>
-<wire x1="12.7" y1="35.56" x2="35.56" y2="35.56" width="0.1524" layer="91"/>
-<wire x1="35.56" y1="35.56" x2="35.56" y2="40.64" width="0.1524" layer="91"/>
-<junction x="35.56" y="40.64"/>
 <pinref part="JSN-SR04T_3" gate="A" pin="4"/>
 <wire x1="-20.32" y1="60.96" x2="-27.94" y2="60.96" width="0.1524" layer="91"/>
@@
 <pinref part="JSN-SR04T_2" gate="A" pin="4"/>
 <wire x1="-40.64" y1="76.2" x2="-40.64" y2="101.6" width="0.1524" layer="91"/>
-</segment>
-</net>
+<pinref part="U$2" gate="G$1" pin="OUT-"/>
+<wire x1="38.1" y1="-2.54" x2="38.1" y2="27.94" width="0.1524" layer="91"/>
+<wire x1="38.1" y1="27.94" x2="132.08" y2="27.94" width="0.1524" layer="91"/>
+</segment>
+</net>
+<net name="N$11" class="0">
+<segment>
+<wire x1="12.7" y1="40.64" x2="12.7" y2="35.56" width="0.1524" layer="91"/>
+</segment>
+</net>
+<net name="N$12" class="0">
+<segment>
+<wire x1="12.7" y1="43.18" x2="12.7" y2="50.8" width="0.1524" layer="91"/>
+</segment>
+</net>
